File: Hardware/RFVD_SENSOR_BOARD_Rev5/RFVD_SENSOR_BOARD.kicad_pcb (KiCad board)
At the start: 6 copper layers, 52 x 90 mm, 341 parts, among them J1 AIMD_IN, J10 TYPE-C-31-M-12, J11 LSHM-120-02.5-L-DV-A-N-K-TR, J2 2053380004, J3 DM3AT-SF-PEJM5, J300 CAL_IN, J4 XF2M-4015-1A, J6 TC2030-NL SWD POGO DNP, J8 84953-6, Q201 AO3401A, Q202 2N7002, Q203 AO3400A, Q301 AO3400A, Q302 2N7002, Q303 AO3401A, SW1 RECORD / STOP, SW2 MARK, SW5 B3U-1000P, U1 TLV809EA46DBZR, U10 TPS2553DDBVR, U11 TMP117AIDRVR, U13 AD7380BCPZ-RL7, U2 ADL5511ACPZ-R7, U3 OPA2320, U301 BQ25798RQMR, U302 BQ29209DRBR, U303 TPS70933DBVR, U304 TPD4E05U06DQAR, U4 OPA2320, U401 TPS2553DDBVR, U402 TPS259631DDAR, U403 TCA9517ADGKR, U5 REF5030IDR, U6 LMR43620MB5RPER, U7 LT3045EMSE#PBF (+5V_A), U701 SHT40-AD1B-R2, U8 STM32H743VIT6, U9 APS6404L-3SQR-SN, U901 EMIF06-MSD02N16, Y1 12MHz 3.3V CMOS, Y2 32.768kHz 7pF

Commit message: TrackingRedo-Rev5
Parts:
- C105, C106, C107, R10, R102, RN201: moved to B.Cu
- C701, D301, R103, U701: moved to F.Cu
- moved TP306 8.75 mm to (122.1, 125.9)
- moved TP305 6.95 mm to (122.1, 129.0)
- moved U304 6.14 mm to (125.1, 127.7), turned to -90 degrees
- moved C20 5.99 mm to (132.7, 76.3)
- moved C301 5.61 mm to (127.9, 130.2), turned to 0 degrees
- moved C107 4.43 mm to (135.5, 84.3), turned to 135 degrees
- moved C106 4.21 mm to (136.7, 86.1), turned to -135 degrees
- moved C15 4.09 mm to (137.7, 78.8), turned to 0 degrees
- moved R12 3.94 mm to (141.0, 76.6), turned to -90 degrees
- moved R100 3.40 mm to (142.1, 80.2)
- moved RN60 3.37 mm to (124.1, 90.8)
- moved R53 3.22 mm to (135.7, 104.5), turned to 180 degrees
- moved C102 3.19 mm to (140.3, 81.3), turned to -45 degrees
- moved C93 2.72 mm to (144.8, 98.6), turned to -90 degrees
- moved R10 2.67 mm to (143.6, 76.4), turned to 180 degrees
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Routing:
- net +3V3_D: track 172.1 -> 48.7 mm, vias 12 -> 8
- net I2C_SCL: track 118.6 -> 3.95 mm, vias 10 -> 3
- net /Expansion mezzanine/EXP_TMR1: track 85.9 -> 2.78 mm, vias 5 -> 1
- net EXP_3V3_EN: track 83.4 -> 1.00 mm, vias 3 -> 1
- net +3V3_UI: track 78.7 -> 0.00 mm, vias 12 -> 0
- net VSYS: track 90.3 -> 12.1 mm, vias 11 -> 2
- net VBUS: track 71.1 -> 4.37 mm, vias 13 -> 0
- net EXP_INT0_N_MCU: track 65.9 -> 0.00 mm, vias 5 -> 0
- net SWCLK: track 62.9 -> 0.15 mm, vias 8 -> 0
- net SWDIO: track 61.4 -> 0.00 mm, vias 4 -> 0
- net +3V3_EXP: track 83.5 -> 26.8 mm, vias 11 -> 0
- net I2C_SDA: track 56.3 -> 1.76 mm, vias 7 -> 3
- net VBAT_PACK: track 53.5 -> 0.00 mm, vias 8 -> 0
- net TP_RST: track 52.2 -> 0.00 mm, vias 2 -> 1
- net EXP_FAULT_N: track 48.1 -> 0.03 mm, vias 6 -> 1
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
Commit message: TrackCheckpoint-Rev5
Parts:
- R412: moved to F.Cu
- moved R412 6.92 mm to (141.5, 131.7)
- moved C405 1.97 mm to (136.1, 119.1), turned to 180 degrees
- moved R426 1.92 mm to (138.7, 125.7), turned to -90 degrees
- moved R438 1.92 mm to (144.0, 137.6), turned to 90 degrees
- moved R414 1.91 mm to (137.6, 137.6), turned to 90 degrees
- moved C403 1.73 mm to (136.2, 137.2), turned to 180 degrees
- moved R437 1.62 mm to (141.9, 137.6)
- moved R425 1.56 mm to (139.7, 139.1), turned to 0 degrees
- moved R440 1.33 mm to (145.5, 137.3), turned to 180 degrees
- moved R423 1.22 mm to (138.7, 137.6)
- moved R436 1.05 mm to (139.8, 137.6), turned to -90 degrees
- moved R104 1.02 mm to (134.5, 86.6), turned to 45 degrees
- moved R441 0.98 mm to (137.6, 125.7)
- moved R103 0.98 mm to (132.1, 85.9), turned to -135 degrees
- moved R407 0.95 mm to (136.1, 120.4)
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Routing:
- net +3V3_EXP: track 26.8 -> 41.0 mm, vias 0 -> 3
- net GND: track 76.0 -> 83.4 mm, vias 396 -> 427
- net /RF input and detector/VRMS_DIAG: track 0.80 -> 8.21 mm
- net EXTADC_SDI: track 0.00 -> 5.77 mm
- net Net-(U3A-+): track 6.17 -> 9.51 mm
- net Net-(U8-PC1): track 2.88 -> 6.18 mm, vias 0 -> 1
- net /Expansion mezzanine/EXP_SPI_CS1_N: track 2.87 -> 5.43 mm
- net +3V3_UI: track 0.00 -> 1.85 mm, vias 0 -> 1
- net /Expansion mezzanine/EXP_INT0_N: track 3.74 -> 5.25 mm
- net /Expansion mezzanine/EXP_SPI_MISO: track 4.76 -> 3.83 mm
- net EXTADC_SDOA: track 3.97 -> 3.06 mm
- net EXTADC_SCLK: track 1.93 -> 2.80 mm
- net /Expansion mezzanine/EXP_IO1: track 3.96 -> 3.19 mm
- net /External ADC/ADC_SDOA_U13: track 2.25 -> 2.98 mm
- net /Expansion mezzanine/EXP_TMR_IN: track 4.16 -> 3.49 mm
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