File: Hardware/RFVD_SENSOR_BOARD_Rev5/RFVD_SENSOR_BOARD.kicad_pcb (KiCad board)
At the start: 6 copper layers, 52 x 90 mm, 341 parts, among them J1 AIMD_IN, J10 TYPE-C-31-M-12, J11 LSHM-120-02.5-L-DV-A-N-K-TR, J2 2053380004, J3 DM3AT-SF-PEJM5, J300 CAL_IN, J4 XF2M-4015-1A, J6 TC2030-NL SWD POGO DNP, J8 84953-6, Q201 AO3401A, Q202 2N7002, Q203 AO3400A, Q301 AO3400A, Q302 2N7002, Q303 AO3401A, SW1 RECORD / STOP, SW2 MARK, SW5 B3U-1000P, U1 TLV809EA46DBZR, U10 TPS2553DDBVR, U11 TMP117AIDRVR, U13 AD7380BCPZ-RL7, U2 ADL5511ACPZ-R7, U3 OPA2320, U301 BQ25798RQMR, U302 BQ29209DRBR, U303 TPS70933DBVR, U304 TPD4E05U06DQAR, U4 OPA2320, U401 TPS2553DDBVR, U402 TPS259631DDAR, U403 TCA9517ADGKR, U5 REF5030IDR, U6 LMR43620MB5RPER, U7 LT3045EMSE#PBF (+5V_A), U701 SHT40-AD1B-R2, U8 STM32H743VIT6, U9 APS6404L-3SQR-SN, U901 EMIF06-MSD02N16, Y1 12MHz 3.3V CMOS, Y2 32.768kHz 7pF

Commit message: TrackCheckpoint2-Rev5
Parts:
- R417: moved to F.Cu
- moved D203 30.3 mm to (159.3, 135.7), turned to -90 degrees
- moved D204 17.5 mm to (147.4, 123.6), turned to 90 degrees
- moved R417 11.8 mm to (141.1, 134.8), turned to -90 degrees
- moved R47 10.5 mm to (139.6, 102.0), turned to -90 degrees
- moved C410 8.24 mm to (149.4, 140.6), turned to -90 degrees
- moved C402 7.45 mm to (151.9, 140.9), turned to 0 degrees
- moved C701 6.28 mm to (155.2, 140.5)
- moved U701 6.15 mm to (156.4, 138.1), turned to 0 degrees
- moved C409 6.13 mm to (156.7, 139.6), turned to 180 degrees
- moved C67 5.31 mm to (143.9, 101.8), turned to 0 degrees
- moved R46 4.18 mm to (143.5, 103.3)
- moved U403 3.98 mm to (151.9, 138.1), turned to 180 degrees
- moved C318 3.43 mm to (140.9, 106.4), turned to 90 degrees
- moved C303 3.09 mm to (148.3, 114.9)
- moved TP302 3.06 mm to (162.8, 125.5)
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Routing:
- net TP_RST: track 0.00 -> 35.2 mm, vias 1 -> 2
- net TP_INT: track 0.00 -> 30.7 mm, vias 0 -> 2
- net LCD_RST: track 0.00 -> 27.7 mm
- net SD_D2_MCU: track 0.00 -> 10.9 mm, vias 0 -> 1
- net +3V3_EXP: track 41.0 -> 51.4 mm, vias 3 -> 6
- net SD_CMD_MCU: track 0.00 -> 10.3 mm, vias 0 -> 1
- net SD_D3_MCU: track 0.00 -> 9.78 mm, vias 0 -> 1
- net VSYS: track 12.1 -> 20.5 mm
- net /Expansion mezzanine/EXP_I2C_SCL: track 2.46 -> 10.7 mm
- net SD_CD_N: track 0.00 -> 8.12 mm, vias 0 -> 1
- net +3V3_D: track 49.0 -> 41.1 mm, vias 8 -> 9
- net SD_CLK_MCU: track 0.00 -> 7.39 mm, vias 0 -> 1
- net /SD and capture memory/SD_D2: track 0.00 -> 4.97 mm, vias 0 -> 1
- net /SD and capture memory/SD_D3: track 0.00 -> 4.47 mm, vias 0 -> 1
- net Net-(Q202-D): track 0.00 -> 4.33 mm, vias 0 -> 1
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